File: epd-boy-2025.kicad_sch (KiCad schematic)
At the start: 39 parts, among them J1 FH12A-24S-0.5SH(55), Q1 SI1308EDL-T1-GE3, SW1 SW_Push, SW10 SW_SPDT, SW2 SW_Push, SW3 SW_Push, SW4 SW_Push, SW5 SW_Push, SW6 SW_Push, SW7 SW_Push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

Commit message: Revision
Parts:
- SW9: footprint Button_Switch_SMD:SW_SPST_CK_KMS2xxG -> Button_Switch_SMD:SW_SPST_CK_KMS2xxGP
- U1: footprint User_Footprints:xiao-ble-smd-cutout-nfc -> Project:xiao-ble-smd-cutout-nfc
Changed lines of the file:
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@@
 			)
 		)
-		(property "Footprint" "User_Footprints:xiao-ble-smd-cutout-nfc"
+		(property "Footprint" "Project:xiao-ble-smd-cutout-nfc"
 			(at 54.61 35.56 0)
 			(effects
@@
 			)
 		)
-		(property "Footprint" "Button_Switch_SMD:SW_SPST_CK_KMS2xxG"
+		(property "Footprint" "Button_Switch_SMD:SW_SPST_CK_KMS2xxGP"
 			(at 68.58 17.78 0)
 			(effects
